Commit message: 完成模拟示教器的初步开发与联调,不过存在控制移动后无法停止的Bug

File: src/data_collect_sim/urdf/fanuc_m20ib25_gz.xacro (robot description, xacro)
@@ -1,10 +1,60 @@
 <?xml version="1.0"?>
 <robot name="fanuc_m20ib25_gz" xmlns:xacro="http://www.ros.org/wiki/xacro">
-  <xacro:arg name="enable_gz_camera_plugins" default="false"/>
+  <xacro:arg name="use_gz_sensors" default="false"/>
+  <xacro:arg name="base_x" default="0.2"/>
+  <xacro:arg name="base_y" default="0.0"/>
+  <xacro:arg name="base_z" default="0.125"/>
+  <xacro:arg name="base_roll" default="0.0"/>
+  <xacro:arg name="base_pitch" default="0.0"/>
+  <xacro:arg name="base_yaw" default="0.0"/>
   <xacro:include filename="$(find data_collect_sim)/urdf/m20ib25_macro.xacro"/>
+  <xacro:macro name="disable_gz_gravity" params="link_name">
+    <gazebo reference="${link_name}">
+      <gravity>false</gravity>
+      <self_collide>false</self_collide>
+    </gazebo>
+  </xacro:macro>
+  <xacro:macro name="gz_joint_position_controller" params="joint_name p_gain cmd_max">
+    <gazebo>
+      <plugin
+        filename="ignition-gazebo-joint-position-controller-system"
+        name="gz::sim::systems::JointPositionController">
+        <joint_name>${joint_name}</joint_name>
+        <topic>/fanuc_m20i/${joint_name}/cmd_pos</topic>
+        <p_gain>${p_gain}</p_gain>
+        <cmd_max>${cmd_max}</cmd_max>
+        <cmd_min>-${cmd_max}</cmd_min>
+        <initial_position>0.0</initial_position>
+      </plugin>
+    </gazebo>
+  </xacro:macro>
   <gazebo>
-    <static>true</static>
+    <static>false</static>
   </gazebo>
+  <link name="world"/>
   <xacro:fanuc_m20ib25 prefix=""/>
+  <joint name="world_base_link" type="fixed">
+    <origin
+      xyz="$(arg base_x) $(arg base_y) $(arg base_z)"
+      rpy="$(arg base_roll) $(arg base_pitch) $(arg base_yaw)"/>
+    <parent link="world"/>
+    <child link="base_link"/>
+  </joint>
+  <xacro:disable_gz_gravity link_name="base_link"/>
+  <xacro:disable_gz_gravity link_name="link_1"/>
+  <xacro:disable_gz_gravity link_name="link_2"/>
+  <xacro:disable_gz_gravity link_name="link_3"/>
+  <xacro:disable_gz_gravity link_name="link_4"/>
+  <xacro:disable_gz_gravity link_name="link_5"/>
+  <xacro:disable_gz_gravity link_name="link_6"/>
+  <xacro:disable_gz_gravity link_name="base"/>
+  <xacro:disable_gz_gravity link_name="flange"/>
+  <xacro:disable_gz_gravity link_name="tool0"/>
+  <xacro:gz_joint_position_controller joint_name="joint_1" p_gain="800" cmd_max="1200"/>
+  <xacro:gz_joint_position_controller joint_name="joint_2" p_gain="900" cmd_max="1400"/>
+  <xacro:gz_joint_position_controller joint_name="joint_3" p_gain="900" cmd_max="1400"/>
+  <xacro:gz_joint_position_controller joint_name="joint_4" p_gain="500" cmd_max="800"/>
+  <xacro:gz_joint_position_controller joint_name="joint_5" p_gain="500" cmd_max="800"/>
+  <xacro:gz_joint_position_controller joint_name="joint_6" p_gain="350" cmd_max="600"/>
   <link name="camera_mount">
     <visual>
@@ -30,12 +80,14 @@
   </link>
   <joint name="tool0_camera_mount" type="fixed">
-    <origin xyz="0.04 0 0.13" rpy="0 0 0"/>
+    <origin xyz="0.04 0 0.13" rpy="0 3.141592653589793 0"/>
     <parent link="tool0"/>
     <child link="camera_mount"/>
   </joint>
-  <xacro:if value="$(arg enable_gz_camera_plugins)">
+  <xacro:disable_gz_gravity link_name="camera_mount"/>
+  <xacro:if value="$(arg use_gz_sensors)">
     <gazebo reference="camera_mount">
       <sensor name="pool_camera_2d" type="camera">
         <pose>0 0 0 0 0 0</pose>
+        <topic>/fanuc_m20i/pool_camera/image</topic>
         <camera>
           <horizontal_fov>1.047</horizontal_fov>
@@ -53,27 +105,23 @@
         <update_rate>30</update_rate>
         <visualize>true</visualize>
-        <plugin name="ros_gz_pool_camera_plugin" filename="libros_gz_camera.so">
-          <ros_topic>/image_topic</ros_topic>
-          <frame_name>camera_mount</frame_name>
-          <qos>sensor_default</qos>
-        </plugin>
       </sensor>
-      <sensor name="line_scan_3d" type="depth">
+      <sensor name="tcp_rgbd" type="rgbd_camera">
         <pose>0 0 0 0 0 0</pose>
-        <depth>
+        <topic>/fanuc_m20i/tcp_rgbd</topic>
+        <camera>
+          <horizontal_fov>1.047</horizontal_fov>
+          <image>
+            <width>640</width>
+            <height>480</height>
+            <format>R8G8B8</format>
+          </image>
           <clip>
             <near>0.1</near>
             <far>30.0</far>
           </clip>
-        </depth>
+        </camera>
         <always_on>true</always_on>
         <update_rate>15</update_rate>
         <visualize>false</visualize>
-        <plugin name="ros_gz_line_scan_plugin" filename="libros_gz_depth_camera.so">
-          <ros_topic>/tcp_depth_image</ros_topic>
-          <pointcloud_topic>/tcp_cloud_raw</pointcloud_topic>
-          <frame_name>camera_mount</frame_name>
-          <qos>sensor_default</qos>
-        </plugin>
       </sensor>
     </gazebo>
