Commit message: 重排项目文件结构,删除荣誉仿真材料模型

File: src/robot_sim_description/macros/gazebo_sensors.xacro (robot description, xacro)
@@ -1,9 +1,9 @@
 <?xml version="1.0"?>
 <robot xmlns:xacro="http://www.ros.org/wiki/xacro">
-  <xacro:macro name="panda_gazebo_sensors" params="prefix enable_camera enable_depth enable_lidar enable_imu">
+  <xacro:macro name="robot_sim_gazebo_sensors" params="prefix enable_camera enable_depth enable_lidar enable_imu camera_pose:='0 0 0 0 0 0' depth_pose:='0 0 0 0 0 0' lidar_2d_pose:='0 0 0.035 0 0 0' lidar_3d_pose:='0 0 0.055 0 0 0' imu_pose:='0 0 0.02 0 0 0'">
     <xacro:if value="${enable_camera}">
       <gazebo reference="${prefix}camera_mount">
         <sensor name="color_camera" type="camera">
-          <pose>0 0 0 0 0 0</pose>
+          <pose>${camera_pose}</pose>
           <topic>/camera/color/image_raw</topic>
           <camera>
@@ -28,5 +28,5 @@
       <gazebo reference="${prefix}camera_mount">
         <sensor name="rgbd_camera" type="rgbd_camera">
-          <pose>0 0 0 0 0 0</pose>
+          <pose>${depth_pose}</pose>
           <topic>/camera/depth</topic>
           <camera>
@@ -51,5 +51,5 @@
       <gazebo reference="${prefix}camera_mount">
         <sensor name="lidar_2d" type="gpu_lidar">
-          <pose>0 0 0.035 0 0 0</pose>
+          <pose>${lidar_2d_pose}</pose>
           <topic>/scan</topic>
           <update_rate>20</update_rate>
@@ -74,5 +74,5 @@
       <gazebo reference="${prefix}camera_mount">
         <sensor name="lidar_3d" type="gpu_lidar">
-          <pose>0 0 0.055 0 0 0</pose>
+          <pose>${lidar_3d_pose}</pose>
           <topic>/lidar</topic>
           <update_rate>10</update_rate>
@@ -105,5 +105,5 @@
       <gazebo reference="${prefix}camera_mount">
         <sensor name="imu" type="imu">
-          <pose>0 0 0.02 0 0 0</pose>
+          <pose>${imu_pose}</pose>
           <topic>/imu/data</topic>
           <always_on>true</always_on>
@@ -114,3 +114,12 @@
     </xacro:if>
   </xacro:macro>
+  <xacro:macro name="panda_gazebo_sensors" params="prefix enable_camera enable_depth enable_lidar enable_imu">
+    <xacro:robot_sim_gazebo_sensors
+      prefix="${prefix}"
+      enable_camera="${enable_camera}"
+      enable_depth="${enable_depth}"
+      enable_lidar="${enable_lidar}"
+      enable_imu="${enable_imu}"
+    />
+  </xacro:macro>
 </robot>

File: src/robot_sim_description/macros/ros2_control.xacro (robot description, xacro)
@@ -14,5 +14,5 @@
     </joint>
   </xacro:macro>
-  <xacro:macro name="panda_ros2_control" params="prefix hardware_plugin controllers_file controller_manager_name use_gz_ros2_control ros_namespace">
+  <xacro:macro name="robot_sim_gazebo_ros2_control_plugin" params="use_gz_ros2_control controllers_file controller_manager_name ros_namespace">
     <xacro:if value="${use_gz_ros2_control}">
       <gazebo>
@@ -28,4 +28,12 @@
       </gazebo>
     </xacro:if>
+  </xacro:macro>
+  <xacro:macro name="panda_ros2_control" params="prefix hardware_plugin controllers_file controller_manager_name use_gz_ros2_control ros_namespace">
+    <xacro:robot_sim_gazebo_ros2_control_plugin
+      use_gz_ros2_control="${use_gz_ros2_control}"
+      controllers_file="${controllers_file}"
+      controller_manager_name="${controller_manager_name}"
+      ros_namespace="${ros_namespace}"
+    />
     <ros2_control name="${prefix}PandaSystem" type="system">
       <hardware>

File: src/robot_sim_description/macros/sensor_mounts.xacro (robot description, xacro)
@@ -1,8 +1,8 @@
 <?xml version="1.0"?>
 <robot xmlns:xacro="http://www.ros.org/wiki/xacro">
-  <xacro:macro name="panda_sensor_mounts" params="prefix camera_mesh">
+  <xacro:macro name="robot_sim_sensor_mounts" params="prefix parent_link joint_name camera_mesh mount_xyz mount_rpy visual_xyz:='0 0 0' visual_rpy:='0 0 0' collision_xyz:='0 0 0' collision_rpy:='0 0 0' frame_xyz:='0 0 0' lidar_2d_xyz:='0 0 0.035' lidar_3d_xyz:='0 0 0.055' imu_xyz:='0 0 0.02'">
     <link name="${prefix}camera_mount">
       <visual>
-        <origin xyz="0 0 0" rpy="0 0 1.5707963267948966"/>
+        <origin xyz="${visual_xyz}" rpy="${visual_rpy}"/>
         <geometry>
           <mesh filename="${camera_mesh}"/>
@@ -10,5 +10,5 @@
       </visual>
       <collision>
-        <origin xyz="0.02 0 0.034" rpy="0 0 1.5707963267948966"/>
+        <origin xyz="${collision_xyz}" rpy="${collision_rpy}"/>
         <geometry>
           <box size="0.165 0.040 0.030"/>
@@ -17,12 +17,12 @@
       <xacro:simple_inertial mass="0.3" ixx="0.0002" iyy="0.0008" izz="0.0008"/>
     </link>
-    <joint name="${prefix}panda_link8_camera_mount" type="fixed">
-      <origin xyz="0.10 0 -0.10" rpy="0 -0.7853981633974483 3.141592653589793"/>
-      <parent link="${prefix}panda_link8"/>
+    <joint name="${prefix}${joint_name}" type="fixed">
+      <origin xyz="${mount_xyz}" rpy="${mount_rpy}"/>
+      <parent link="${prefix}${parent_link}"/>
       <child link="${prefix}camera_mount"/>
     </joint>
     <link name="${prefix}camera_color_frame"/>
     <joint name="${prefix}camera_color_frame_joint" type="fixed">
-      <origin xyz="0 0 0" rpy="0 0 0"/>
+      <origin xyz="${frame_xyz}" rpy="0 0 0"/>
       <parent link="${prefix}camera_mount"/>
       <child link="${prefix}camera_color_frame"/>
@@ -30,5 +30,5 @@
     <link name="${prefix}rgbd_camera_frame"/>
     <joint name="${prefix}rgbd_camera_frame_joint" type="fixed">
-      <origin xyz="0 0 0" rpy="0 0 0"/>
+      <origin xyz="${frame_xyz}" rpy="0 0 0"/>
       <parent link="${prefix}camera_mount"/>
       <child link="${prefix}rgbd_camera_frame"/>
@@ -36,5 +36,5 @@
     <link name="${prefix}lidar_2d_frame"/>
     <joint name="${prefix}lidar_2d_frame_joint" type="fixed">
-      <origin xyz="0 0 0.035" rpy="0 0 0"/>
+      <origin xyz="${lidar_2d_xyz}" rpy="0 0 0"/>
       <parent link="${prefix}camera_mount"/>
       <child link="${prefix}lidar_2d_frame"/>
@@ -42,5 +42,5 @@
     <link name="${prefix}lidar_3d_frame"/>
     <joint name="${prefix}lidar_3d_frame_joint" type="fixed">
-      <origin xyz="0 0 0.055" rpy="0 0 0"/>
+      <origin xyz="${lidar_3d_xyz}" rpy="0 0 0"/>
       <parent link="${prefix}camera_mount"/>
       <child link="${prefix}lidar_3d_frame"/>
@@ -48,8 +48,22 @@
     <link name="${prefix}imu_link"/>
     <joint name="${prefix}imu_joint" type="fixed">
-      <origin xyz="0 0 0.02" rpy="0 0 0"/>
+      <origin xyz="${imu_xyz}" rpy="0 0 0"/>
       <parent link="${prefix}camera_mount"/>
       <child link="${prefix}imu_link"/>
     </joint>
   </xacro:macro>
+  <xacro:macro name="panda_sensor_mounts" params="prefix camera_mesh">
+    <xacro:robot_sim_sensor_mounts
+      prefix="${prefix}"
+      parent_link="panda_link8"
+      joint_name="panda_link8_camera_mount"
+      camera_mesh="${camera_mesh}"
+      mount_xyz="0.10 0 -0.10"
+      mount_rpy="0 -0.7853981633974483 3.141592653589793"
+      visual_xyz="0 0 0"
+      visual_rpy="0 0 1.5707963267948966"
+      collision_xyz="0.02 0 0.034"
+      collision_rpy="0 0 1.5707963267948966"
+    />
+  </xacro:macro>
 </robot>

File: src/robot_sim_description/robots/panda.urdf.xacro (robot description, xacro)
@@ -9,6 +9,6 @@
   <xacro:arg name="controllers_file" default=""/>
   <xacro:arg name="controller_manager_name" default="controller_manager"/>
-  <xacro:arg name="mesh_root" default="package://robot_sim_description/models/panda_arm/meshes"/>
-  <xacro:arg name="camera_mesh" default="package://robot_sim_description/models/rgbd_camera/meshes/3dCamera.DAE"/>
+  <xacro:arg name="mesh_root" default="package://robot_sim_description/models/robots/panda/meshes"/>
+  <xacro:arg name="camera_mesh" default="package://robot_sim_description/models/sensors/cameras/rgbd_camera/meshes/3dCamera.DAE"/>
   <xacro:arg name="use_gz_ros2_control" default="false"/>
   <xacro:arg name="ros_namespace" default=""/>
